Commit message: Remove "virtual_" prefix from joints and links

File: urdf/wrist.transmissions.xacro (robot description, xacro)
@@ -2,10 +2,10 @@
 <robot xmlns:xacro="http://www.ros.org/wiki/xacro">
   <xacro:macro name="wrist_transmission" params="axes">
-    <transmission name="virtual_${axes}_transmission">
+    <transmission name="${axes}_transmission">
       <type>transmission_interface/SimpleTransmission</type>
-      <joint name="virtual_${axes}_joint">
+      <joint name="${axes}_joint">
         <hardwareInterface>hardware_interface/EffortJointInterface</hardwareInterface>
       </joint>
-      <actuator name="virtual_${axes}_joint_motor">
+      <actuator name="${axes}_joint_motor">
         <hardwareInterface>hardware_interface/EffortJointInterface</hardwareInterface>
         <mechanicalReduction>1</mechanicalReduction>

File: urdf/wrist.urdf.xacro (robot description, xacro)
@@ -15,13 +15,13 @@
     <!-- links and joints for translation -->
     <link name="world"/>
-    <joint name="virtual_px_joint" type="prismatic">
+    <joint name="px_joint" type="prismatic">
         <origin rpy="0 0 0" xyz="0 0 0"/>
         <axis xyz="1 0 0"/>
         <parent link="world"/>
-        <child link="virtual_px_link"/>
+        <child link="px_link"/>
         <limit effort="${translation_effort}" lower="${translation_low_lim}" upper="${translation_up_lim}" velocity="${translation_velocity}"/>
         <dynamics damping="${translation_damping}" friction="${translation_friction}"/>
     </joint>
-    <link name="virtual_px_link">
+    <link name="px_link">
         <inertial>
             <origin rpy="0 0 0" xyz="0 0 0"/>
@@ -30,13 +30,13 @@
         </inertial>
     </link>
-    <joint name="virtual_py_joint" type="prismatic">
+    <joint name="py_joint" type="prismatic">
         <origin rpy="0 0 0" xyz="0 0 0"/>
         <axis xyz="0 1 0"/>
-        <parent link="virtual_px_link"/>
-        <child link="virtual_py_link"/>
+        <parent link="px_link"/>
+        <child link="py_link"/>
         <limit effort="${translation_effort}" lower="${translation_low_lim}" upper="${translation_up_lim}" velocity="${translation_velocity}"/>
         <dynamics damping="${translation_damping}" friction="${translation_friction}"/>
     </joint>
-    <link name="virtual_py_link">
+    <link name="py_link">
         <inertial>
             <origin rpy="0 0 0" xyz="0 0 0"/>
@@ -45,13 +45,13 @@
         </inertial>
     </link>
-    <joint name="virtual_pz_joint" type="prismatic">
+    <joint name="pz_joint" type="prismatic">
         <origin rpy="0 0 0" xyz="0 0 0"/>
         <axis xyz="0 0 1"/>
-        <parent link="virtual_py_link"/>
-        <child link="virtual_pz_link"/>
+        <parent link="py_link"/>
+        <child link="pz_link"/>
         <limit effort="${translation_effort}" lower="${translation_low_lim}" upper="${translation_up_lim}" velocity="${translation_velocity}"/>
         <dynamics damping="${translation_damping}" friction="${translation_friction}"/>
     </joint>
-    <link name="virtual_pz_link">
+    <link name="pz_link">
         <inertial>
             <origin rpy="0 0 0" xyz="0 0 0"/>
@@ -61,13 +61,13 @@
     </link>
     <!-- links and joints for rotation -->
-    <joint name="virtual_ry_joint" type="continuous">
+    <joint name="ry_joint" type="continuous">
         <origin rpy="0 0 0" xyz="0 0 0"/>
         <axis xyz="0 0 1"/>
-        <parent link="virtual_pz_link"/>
-        <child link="virtual_ry_link"/>
+        <parent link="pz_link"/>
+        <child link="ry_link"/>
         <limit effort="${rotation_effort}" velocity="${rotation_velocity}"/>
         <dynamics damping="${rotation_damping}" friction="${rotation_friction}"/>
     </joint>
-    <link name="virtual_ry_link">
+    <link name="ry_link">
         <inertial>
             <origin rpy="0 0 0" xyz="0 0 0"/>
@@ -76,13 +76,13 @@
         </inertial>
     </link>
-    <joint name="virtual_rp_joint" type="continuous">
+    <joint name="rp_joint" type="continuous">
         <origin rpy="0 0 0" xyz="0 0 0"/>
         <axis xyz="0 1 0"/>
-        <parent link="virtual_ry_link"/>
-        <child link="virtual_rp_link"/>
+        <parent link="ry_link"/>
+        <child link="rp_link"/>
         <limit effort="${rotation_effort}" velocity="${rotation_velocity}"/>
         <dynamics damping="${rotation_damping}" friction="${rotation_friction}"/>
     </joint>
-    <link name="virtual_rp_link">
+    <link name="rp_link">
         <inertial>
             <origin rpy="0 0 0" xyz="0 0 0"/>
@@ -92,8 +92,8 @@
     </link>
     <!-- if you want to use this package with other robot hands, simply replace the "shell" link with the base link of your robot hand -->
-    <joint name="virtual_rr_joint" type="continuous">
+    <joint name="rr_joint" type="continuous">
         <origin rpy="0 0 0" xyz="0 0 0"/>
         <axis xyz="1 0 0"/>
-        <parent link="virtual_rp_link"/>
+        <parent link="rp_link"/>
         <child link="shell"/>
         <limit effort="${rotation_effort}" velocity="${rotation_velocity}"/>
