Commit message: Outsource inertia values

File: urdf/wrist.urdf.xacro (robot description, xacro)
@@ -1,4 +1,6 @@
 <?xml version="1.0" ?>
-<robot xmlns:xacro="http://www.ros.org/wiki/xacro" name="reflex">
+<robot xmlns:xacro="http://www.ros.org/wiki/xacro">
+    <!-- name of base link of your robotic hand -->
+    <xacro:arg name="base_link_name" default="base_link"/>
     <!-- translation properties -->
     <xacro:property name="translation_effort" value="1000"/>
@@ -13,4 +15,12 @@
     <xacro:property name="rotation_damping" value="60"/>
     <xacro:property name="rotation_friction" value="0"/>
+    <!-- link properties -->
+    <xacro:property name="mass" value="1"/>
+    <xacro:property name="ixx" value="0.01"/>
+    <xacro:property name="ixy" value="0"/>
+    <xacro:property name="ixz" value="0"/>
+    <xacro:property name="iyy" value="0.01"/>
+    <xacro:property name="iyz" value="0"/>
+    <xacro:property name="izz" value="0.01"/>
     <!-- links and joints for translation -->
     <link name="world"/>
@@ -26,6 +36,6 @@
         <inertial>
             <origin rpy="0 0 0" xyz="0 0 0"/>
-            <mass value="1"/>
-            <inertia ixx="0.01" ixy="0" ixz="0" iyy="0.01" iyz="0" izz="0.01"/>
+            <mass value="${mass}"/>
+            <inertia ixx="${ixx}" ixy="${ixy}" ixz="${ixz}" iyy="${iyy}" iyz="${iyz}" izz="${izz}"/>
         </inertial>
     </link>
@@ -41,6 +51,6 @@
         <inertial>
             <origin rpy="0 0 0" xyz="0 0 0"/>
-            <mass value="1"/>
-            <inertia ixx="0.01" ixy="0" ixz="0" iyy="0.01" iyz="0" izz="0.01"/>
+            <mass value="${mass}"/>
+            <inertia ixx="${ixx}" ixy="${ixy}" ixz="${ixz}" iyy="${iyy}" iyz="${iyz}" izz="${izz}"/>
         </inertial>
     </link>
@@ -56,6 +66,6 @@
         <inertial>
             <origin rpy="0 0 0" xyz="0 0 0"/>
-            <mass value="1"/>
-            <inertia ixx="0.01" ixy="0" ixz="0" iyy="0.01" iyz="0" izz="0.01"/>
+            <mass value="${mass}"/>
+            <inertia ixx="${ixx}" ixy="${ixy}" ixz="${ixz}" iyy="${iyy}" iyz="${iyz}" izz="${izz}"/>
         </inertial>
     </link>
@@ -72,6 +82,6 @@
         <inertial>
             <origin rpy="0 0 0" xyz="0 0 0"/>
-            <mass value="1"/>
-            <inertia ixx="0.01" ixy="0" ixz="0" iyy="0.01" iyz="0" izz="0.01"/>
+            <mass value="${mass}"/>
+            <inertia ixx="${ixx}" ixy="${ixy}" ixz="${ixz}" iyy="${iyy}" iyz="${iyz}" izz="${izz}"/>
         </inertial>
     </link>
@@ -87,14 +97,13 @@
         <inertial>
             <origin rpy="0 0 0" xyz="0 0 0"/>
-            <mass value="1"/>
-            <inertia ixx="0.01" ixy="0" ixz="0" iyy="0.01" iyz="0" izz="0.01"/>
+            <mass value="${mass}"/>
+            <inertia ixx="${ixx}" ixy="${ixy}" ixz="${ixz}" iyy="${iyy}" iyz="${iyz}" izz="${izz}"/>
         </inertial>
     </link>
-    <!-- if you want to use this package with other robot hands, simply replace the "shell" link with the base link of your robot hand -->
     <joint name="rr_joint" type="continuous">
         <origin rpy="0 0 0" xyz="0 0 0"/>
         <axis xyz="1 0 0"/>
         <parent link="rp_link"/>
-        <child link="shell"/>
+        <child link="$(arg base_link_name)"/>
         <limit effort="${rotation_effort}" velocity="${rotation_velocity}"/>
         <dynamics damping="${rotation_damping}" friction="${rotation_friction}"/>

Commit message: Reduce joint velocities

File: urdf/wrist.urdf.xacro (robot description, xacro)
@@ -5,5 +5,5 @@
     <!-- translation properties -->
     <xacro:property name="translation_effort" value="1000"/>
-    <xacro:property name="translation_velocity" value="0.5"/>
+    <xacro:property name="translation_velocity" value="0.05"/>
     <xacro:property name="translation_up_lim" value="5"/>
     <xacro:property name="translation_low_lim" value="-5"/>
@@ -12,5 +12,5 @@
     <!-- rotation properties -->
     <xacro:property name="rotation_effort" value="1000"/>
-    <xacro:property name="rotation_velocity" value="0.1"/>
+    <xacro:property name="rotation_velocity" value="0.01"/>
     <xacro:property name="rotation_damping" value="60"/>
     <xacro:property name="rotation_friction" value="0"/>

Commit message: Add z lower bound of 0

File: urdf/wrist.urdf.xacro (robot description, xacro)
@@ -8,4 +8,5 @@
     <xacro:property name="translation_up_lim" value="5"/>
     <xacro:property name="translation_low_lim" value="-5"/>
+    <xacro:property name="translation_low_lim_z" value="0"/>
     <xacro:property name="translation_damping" value="60"/>
     <xacro:property name="translation_friction" value="0"/>
@@ -60,5 +61,5 @@
         <parent link="py_link"/>
         <child link="pz_link"/>
-        <limit effort="${translation_effort}" lower="${translation_low_lim}" upper="${translation_up_lim}" velocity="${translation_velocity}"/>
+        <limit effort="${translation_effort}" lower="${translation_low_lim_z}" upper="${translation_up_lim}" velocity="${translation_velocity}"/>
         <dynamics damping="${translation_damping}" friction="${translation_friction}"/>
     </joint>

Commit message: Change lower z limit

File: urdf/wrist.urdf.xacro (robot description, xacro)
@@ -8,5 +8,5 @@
     <xacro:property name="translation_up_lim" value="5"/>
     <xacro:property name="translation_low_lim" value="-5"/>
-    <xacro:property name="translation_low_lim_z" value="0"/>
+    <xacro:property name="translation_low_lim_z" value="-1"/>
     <xacro:property name="translation_damping" value="60"/>
     <xacro:property name="translation_friction" value="0"/>
